File: RFC-Pi-Simple-Hat/RFC-Pi-Simple-Hat.kicad_pcb (KiCad board)
At the start: 2 copper layers, 51 x 55.5 mm, 13 parts, among them J1 sabertooth, J10 spi_1, J11 Barrel_Jack_Switch, J12 Raspberry_Pi_2_3, J2 3V3_0, J3 3V3_1, J4 i2c_0, J5 i2c_1, J6 3V3_2, J7 3V3_3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

Commit message: Updated board
Parts:
- J11: footprint Connector_BarrelJack:BarrelJack_GCT_DCJ200-10-A_Horizontal -> DC-005:NINIGI_DC-005
- J12: moved to B.Cu
- moved J12 2.54 mm to (103.5, 97.0), turned to 0 degrees
- moved J11 2.32 mm to (117.0, 93.5), turned to 90 degrees
Other:
- board text added: "Robotic Football Club 2024 - 25 &.P"
- board text removed: "W.I.P - Andres Perez"
