File: RFC-Pi-Simple-Hat/RFC-Pi-Simple-Hat.kicad_sch (KiCad schematic)
At the start: 12 parts, among them J1 sabertooth, J10 spi_1, J11 Barrel_Jack_Switch, J12 Raspberry_Pi_2_3, J2 3V3_0, J3 3V3_1, J4 i2c_0, J5 i2c_1, J6 3V3_2, J7 3V3_3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

Commit message: Updated board
Parts:
- J1, J2, J4, J5, J6, J7, J8: LCSC Part # (none) -> C234181; now left out of the parts list
- J10, J9: LCSC Part # (none) -> C164168; now left out of the parts list
- J11: footprint Connector_BarrelJack:BarrelJack_GCT_DCJ200-10-A_Horizontal -> DC-005:NINIGI_DC-005; LCSC Part # (none) -> C130239; now left out of the parts list
- J12: JLCPCB Part # C132132 -> (none); LCSC Part # (none) -> C132132; Rotation Offset (none) -> -90; now left out of the parts list
- J3: LCSC Part # (none) -> C234181
